File: Minibadge Devboard.kicad_sch (KiCad schematic)
At the start: 41 parts, among them J1 External power, J2 External switch, SW1 Power, SW3 SPEED, SW4 NTC

Commit message: Fix SW1
Connections:
- net VDD: now also SW1.3 (C)
- no-connect marks 11 -> 10
Other:
- moved on the sheet: R7, SW3, SW4
Changed lines of the file:
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@@
 		(exclude_from_sim no)
 		(at 158.75 99.06 0)
-		(size 44.45 54.61)
+		(size 44.45 58.42)
 		(margins 0.9525 0.9525 0.9525 0.9525)
 		(stroke
@@
 	)
 	(no_connect
-		(at 190.5 114.3)
-	)
-	(no_connect
 		(at 100.33 156.21)
 	)
@@
 	(wire
 		(pts
+			(xy 193.04 115.57) (xy 190.5 115.57)
+		)
+		(stroke
+			(width 0)
+			(type default)
+		)
+	)
+	(wire
+		(pts
 			(xy 134.62 86.36) (xy 137.16 86.36)
 		)
@@
 	(wire
 		(pts
+			(xy 190.5 115.57) (xy 190.5 114.3)
+		)
+		(stroke
+			(width 0)
+			(type default)
+		)
+	)
+	(wire
+		(pts
 			(xy 67.31 91.44) (xy 67.31 93.98)
 		)
@@
 	(wire
 		(pts
-			(xy 166.37 147.32) (xy 168.91 147.32)
+			(xy 166.37 151.13) (xy 168.91 151.13)
 		)
 		(stroke
@@
 	(global_label "FAST"
 		(shape input)
-		(at 173.99 127 180)
+		(at 173.99 130.81 180)
 		(fields_autoplaced yes)
 		(effects
@@
 		)
 		(property "Intersheetrefs" "${INTERSHEET_REFS}"
-			(at 165.9853 127 0)
+			(at 165.9853 130.81 0)
 			(effects
 				(font
@@
 	(global_label "TS"
 		(shape output)
-		(at 184.15 144.78 0)
+		(at 184.15 148.59 0)
 		(fields_autoplaced yes)
 		(effects
@@
 		)
 		(property "Intersheetrefs" "${INTERSHEET_REFS}"
-			(at 189.3123 144.78 0)
+			(at 189.3123 148.59 0)
 			(effects
 				(font
@@
 	(global_label "CLK_LOW"
 		(shape output)
-		(at 184.15 129.54 0)
+		(at 184.15 133.35 0)
 		(fields_autoplaced yes)
 		(effects
@@
 		)
 		(property "Intersheetrefs" "${INTERSHEET_REFS}"
-			(at 195.4809 129.54 0)
+			(at 195.4809 133.35 0)
 			(effects
 				(font
@@
 	(global_label "SLOW"
 		(shape input)
-		(at 173.99 132.08 180)
+		(at 173.99 135.89 180)
 		(fields_autoplaced yes)
 		(effects
@@
 		)
 		(property "Intersheetrefs" "${INTERSHEET_REFS}"
-			(at 166.6505 132.08 0)
+			(at 166.6505 135.89 0)
 			(effects
 				(font
@@
 	(global_label "NTC"
 		(shape input)
-		(at 173.99 142.24 180)
+		(at 173.99 146.05 180)
 		(fields_autoplaced yes)
 		(effects
@@
 		)
 		(property "Intersheetrefs" "${INTERSHEET_REFS}"
-			(at 167.4367 142.24 0)
+			(at 167.4367 146.05 0)
 			(effects
 				(font
@@
 	)
 	(symbol
+		(lib_id "power:VDD")
+		(at 193.04 115.57 0)
+		(unit 1)
+		(exclude_from_sim no)
+		(in_bom yes)
+		(on_board yes)
+		(dnp no)
+		(property "Reference" "#PWR026"
+			(at 193.04 119.38 0)
+			(effects
+				(font
+					(size 1.27 1.27)
+				)
+				(hide yes)
+			)
+		)
+		(property "Value" "VDD"
+			(at 193.04 111.76 0)
+			(effects
+				(font
+					(size 1.27 1.27)
+				)
+			)
+		)
+		(property "Footprint" ""
+			(at 193.04 115.57 0)
+			(effects
+				(font
+					(size 1.27 1.27)
+				)
+				(hide yes)
+			)
+		)
+		(property "Datasheet" ""
+			(at 193.04 115.57 0)
+			(effects
+				(font
+					(size 1.27 1.27)
+				)
+				(hide yes)
+			)
+		)
+		(property "Description" "Power symbol creates a global label with name \"VDD\""
+			(at 193.04 115.57 0)
+			(effects
+				(font
+					(size 1.27 1.27)
+				)
+				(hide yes)
+			)
+		)
+		(pin "1"
+		)
+		(instances
+			(project "Minibadge Devboard"
+				(path "/5e8d5e65-6836-49cf-87c9-8c3c5b8fcf7b"
+					(reference "#PWR026")
+					(unit 1)
+				)
+			)
+		)
+	)
+	(symbol
 		(lib_id "Device:NetTie_2")
 		(at 142.24 57.15 0)
@@
 	(symbol
 		(lib_id "Switch:SW_SPDT")
-		(at 179.07 129.54 180)
+		(at 179.07 133.35 180)
 		(unit 1)
 		(exclude_from_sim no)
@@
 		(fields_autoplaced yes)
 		(property "Reference" "SW3"
-			(at 179.07 120.65 0)
+			(at 179.07 124.46 0)
 			(effects
 				(font
@@
 		)
 		(property "Value" "SPEED"
-			(at 179.07 123.19 0)
+			(at 179.07 127 0)
 			(effects
 				(font
@@
 		)
 		(property "Footprint" "Jumper:SolderJumper-3_P1.3mm_Open_RoundedPad1.0x1.5mm_NumberLabels"
-			(at 179.07 129.54 0)
+			(at 179.07 133.35 0)
 			(effects
 				(font
@@
 		)
 		(property "Datasheet" "~"
-			(at 179.07 121.92 0)
+			(at 179.07 125.73 0)
 			(effects
 				(font
@@
 		)
 		(property "Description" "Switch, single pole double throw"
-			(at 179.07 129.54 0)
+			(at 179.07 133.35 0)
 			(effects
 				(font
@@
 		)
 		(property "LCSC Part #" "C5149822"
-			(at 179.07 129.54 0)
+			(at 179.07 133.35 0)
 			(effects
 				(font
@@
 	(symbol
 		(lib_id "Device:R_Small")
-		(at 171.45 147.32 270)
+		(at 171.45 151.13 270)
 		(mirror x)
 		(unit 1)
@@
 		(dnp no)
 		(property "Reference" "R7"
-			(at 171.45 149.352 90)
+			(at 171.45 153.162 90)
 			(effects
 				(font
@@
 		)
 		(property "Value" "10kΩ"
-			(at 171.45 151.13 90)
+			(at 171.45 154.94 90)
 			(effects
 				(font
@@
 		)
 		(property "Footprint" "Resistor_SMD:R_0603_1608Metric"
-			(at 171.45 147.32 0)
+			(at 171.45 151.13 0)
 			(effects
 				(font
@@
 		)
 		(property "Datasheet" "~"
-			(at 171.45 147.32 0)
+			(at 171.45 151.13 0)
 			(effects
 				(font
@@
 		)
 		(property "Description" "Resistor, small symbol"
-			(at 171.45 147.32 0)
+			(at 171.45 151.13 0)
 			(effects
 				(font
@@
 		)
 		(property "Sim.Type" ""
-			(at 171.45 147.32 90)
+			(at 171.45 151.13 90)
 			(effects
 				(font
@@
 		)
 		(property "LCSC Part #" "C25804"
-			(at 171.45 147.32 90)
+			(at 171.45 151.13 90)
 			(effects
 				(font
@@
 	(symbol
 		(lib_id "power:GND")
-		(at 166.37 147.32 0)
+		(at 166.37 151.13 0)
 		(unit 1)
 		(exclude_from_sim no)
@@
 		(dnp no)
 		(property "Reference" "#PWR023"
-			(at 166.37 153.67 0)
+			(at 166.37 157.48 0)
 			(effects
 				(font
@@
 		)
 		(property "Value" "GND"
-			(at 166.37 151.384 0)
+			(at 166.37 155.194 0)
 			(effects
 				(font
@@
 		)
 		(property "Footprint" ""
-			(at 166.37 147.32 0)
+			(at 166.37 151.13 0)
 			(effects
 				(font
@@
 		)
 		(property "Datasheet" ""
-			(at 166.37 147.32 0)
+			(at 166.37 151.13 0)
 			(effects
 				(font
@@
 		)
 		(property "Description" "Power symbol creates a global label with name \"GND\" , ground"
-			(at 166.37 147.32 0)
+			(at 166.37 151.13 0)
 			(effects
 				(font
@@
 	(symbol
 		(lib_id "Switch:SW_SPDT")
-		(at 179.07 144.78 180)
+		(at 179.07 148.59 180)
 		(unit 1)
 		(exclude_from_sim no)
@@
 		(fields_autoplaced yes)
 		(property "Reference" "SW4"
-			(at 179.07 135.89 0)
+			(at 179.07 139.7 0)
 			(effects
 				(font
@@
 		)
 		(property "Value" "NTC"
-			(at 179.07 138.43 0)
+			(at 179.07 142.24 0)
 			(effects
 				(font
@@
 		)
 		(property "Footprint" "Jumper:SolderJumper-3_P1.3mm_Open_RoundedPad1.0x1.5mm_NumberLabels"
-			(at 179.07 144.78 0)
+			(at 179.07 148.59 0)
 			(effects
 				(font
@@
 		)
 		(property "Datasheet" "~"
-			(at 179.07 137.16 0)
+			(at 179.07 140.97 0)
 			(effects
 				(font
@@
 		)
 		(property "Description" "Switch, single pole double throw"
-			(at 179.07 144.78 0)
+			(at 179.07 148.59 0)
 			(effects
 				(font
@@
 		)
 		(property "LCSC Part #" "C5149822"
-			(at 179.07 144.78 0)
+			(at 179.07 148.59 0)
 			(effects
 				(font

Commit message: update PDF
Parts:
- added R13: 1MΩ, Resistor_SMD:R_0603_1608Metric, symbol Device:R_Small
Connections:
- net GND: now also R8.1; no longer R8.2
- net SW1: now also R8.2, SW1.3 (C); no longer PMOS1.1 (G), SW1.1 (B)
- net SW2: now also PMOS1.1 (G), R13.1; no longer R8.1
- net VDD: now also R13.2; no longer SW1.3 (C)
- no-connect marks 10 -> 11
Other:
- note added: "off"
- note added: "on"
- moved on the sheet: PMOS1, R7, R8, SW1, SW3, SW4
